File: hardware/OBD_CAN_ESP32_V2/OBD_CAN_ESP32_V2.kicad_sch (KiCad schematic)
At the start: 35 parts, among them J1 OBD-II INPUT, J3 ESP32_S3_DEVKITC_J1, J4 ESP32_S3_DEVKITC_J3, Q1 Q_PMOS_GDS, U1 SN65HVD230, U2 TPS54360BDDA

Commit message: hardware: V2 ERC 수정 — 고아 배선 4개 삭제, VBAT_PROTECTED에 PWR_FLAG 추가
Co-Authored-By: Claude Fable 5 <noreply@anthropic.com>
Claude-Session: https://claude.ai/code/session_015Lj2iN8K2AKiUuQKmtXaeP
Changed lines of the file:
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@@
 	(wire
 		(pts
-			(xy 144.78 83.82) (xy 158.75 83.82)
-		)
-		(stroke
-			(width 0)
-			(type default)
-		)
-	)
-	(wire
-		(pts
 			(xy 19.05 40.64) (xy 33.02 40.64)
 		)
@@
 	(wire
 		(pts
-			(xy 144.78 91.44) (xy 158.75 91.44)
-		)
-		(stroke
-			(width 0)
-			(type default)
-		)
-	)
-	(wire
-		(pts
 			(xy 118.11 139.7) (xy 132.08 139.7)
 		)
@@
 	(wire
 		(pts
-			(xy 144.78 88.9) (xy 158.75 88.9)
-		)
-		(stroke
-			(width 0)
-			(type default)
-		)
-	)
-	(wire
-		(pts
 			(xy 38.1 52.07) (xy 38.1 58.42)
 		)
@@
 	(wire
 		(pts
-			(xy 144.78 86.36) (xy 158.75 86.36)
-		)
-		(stroke
-			(width 0)
-			(type default)
-		)
-	)
-	(wire
-		(pts
 			(xy 29.21 163.83) (xy 33.02 163.83)
 		)
@@
 		)
 	)
-	(label "+5V"
-		(at 144.78 88.9 0)
-		(effects
-			(font
-				(size 1.27 1.27)
-			)
-			(justify left bottom)
-		)
-	)
 	(label "+3V3"
 		(at 107.95 119.38 0)
@@
 	)
 	(label "SIGNAL_GND"
-		(at 144.78 86.36 0)
-		(effects
-			(font
-				(size 1.27 1.27)
-			)
-			(justify left bottom)
-		)
-	)
-	(label "SIGNAL_GND"
 		(at 107.95 160.02 0)
 		(effects
@@
 		)
 	)
-	(label "SIGNAL_GND"
-		(at 144.78 91.44 0)
-		(effects
-			(font
-				(size 1.27 1.27)
-			)
-			(justify left bottom)
-		)
-	)
 	(label "CAN_H"
 		(at 217.17 142.24 0)
@@
 		)
 	)
-	(label "VBAT_PROTECTED"
-		(at 144.78 83.82 0)
-		(effects
-			(font
-				(size 1.27 1.27)
-			)
-			(justify left bottom)
-		)
-	)
 	(label "+3V3"
 		(at 33.02 163.83 0)
@@
 		)
 	)
+	(junction
+		(at 287.02 50.8)
+		(diameter 0)
+		(color 0 0 0 0)
+	)
+(symbol
+		(lib_id "power:PWR_FLAG")
+		(at 287.02 50.8 0)
+		(unit 1)
+		(body_style 1)
+		(exclude_from_sim no)
+		(in_bom yes)
+		(on_board yes)
+		(in_pos_files yes)
+		(dnp no)
+		(fields_autoplaced yes)
+		(property "Reference" "#FLG03"
+			(at 287.02 48 0)
+			(hide yes)
+			(show_name no)
+			(do_not_autoplace no)
+			(effects
+				(font
+					(size 1.27 1.27)
+				)
+			)
+		)
+		(property "Value" "PWR_FLAG"
+			(at 287.02 48 90)
+			(show_name no)
+			(do_not_autoplace no)
+			(effects
+				(font
+					(size 1.27 1.27)
+				)
+				(justify left)
+			)
+		)
+		(property "Footprint" ""
+			(at 287.02 48 0)
+			(hide yes)
+			(show_name no)
+			(do_not_autoplace no)
+			(effects
+				(font
+					(size 1.27 1.27)
+				)
+			)
+		)
+		(property "Datasheet" ""
+			(at 287.02 48 0)
+			(hide yes)
+			(show_name no)
+			(do_not_autoplace no)
+			(effects
+				(font
+					(size 1.27 1.27)
+				)
+			)
+		)
+		(property "Description" "Special symbol for telling ERC where power comes from"
+			(at 287.02 48 0)
+			(hide yes)
+			(show_name no)
+			(do_not_autoplace no)
+			(effects
+				(font
+					(size 1.27 1.27)
+				)
+			)
+		)
+		(pin "1"
+		)
+		(instances
+			(project "OBD_CAN_ESP32_V1"
+				(path "/d818bd00-b54e-48fd-8a08-8c2bd25151ea"
+					(reference "#FLG03")
+					(unit 1)
+				)
+			)
+		)
+	)
