File: hardware/OBD_CAN_ESP32_V2/OBD_CAN_ESP32_V2.kicad_sch (KiCad schematic)
At the start: 35 parts, among them J1 OBD-II INPUT, J3 ESP32_S3_DEVKITC_J1, J4 ESP32_S3_DEVKITC_J3, Q1 Q_PMOS_GDS, U1 SN65HVD230, U2 TPS54360BDDA

Commit message: hardware: V2 라이브러리 등록 + 풋프린트 확정 (SWPA6045S, HSOP-8 ThermalVias)
Co-Authored-By: Claude Fable 5 <noreply@anthropic.com>
Claude-Session: https://claude.ai/code/session_015Lj2iN8K2AKiUuQKmtXaeP
Parts:
- L1: footprint Inductor_SMD:L_6.3x6.3_H4.5 -> Inductor_SMD:L_Sunlord_SWPA6045S
- U2: footprint Package_SO:HSOP-8-1EP_3.9x4.9mm_P1.27mm_EP2.41x3.1mm -> Package_SO:HSOP-8-1EP_3.9x4.9mm_P1.27mm_EP2.41x3.1mm_ThermalVias
Changed lines of the file:
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@@
 			)
 		)
-		(property "Footprint" "Inductor_SMD:L_6.3x6.3_H4.5"
+		(property "Footprint" "Inductor_SMD:L_Sunlord_SWPA6045S"
 			(at 340.36 53.34 0)
 			(hide yes)
@@
 			)
 		)
-		(property "Footprint" "Package_SO:HSOP-8-1EP_3.9x4.9mm_P1.27mm_EP2.41x3.1mm"
+		(property "Footprint" "Package_SO:HSOP-8-1EP_3.9x4.9mm_P1.27mm_EP2.41x3.1mm_ThermalVias"
 			(at 312.42 55.88 0)
 			(hide yes)
