File: hardware/OBD_CAN_ESP32_V2/OBD_CAN_ESP32_V2.kicad_sch (KiCad schematic)
At the start: 35 parts, among them J1 OBD-II INPUT, J3 ESP32_S3_DEVKITC_J1, J4 ESP32_S3_DEVKITC_J3, Q1 Q_PMOS_GDS, U1 SN65HVD230, U2 TPS54360BDDA

Commit message: 안테나 구리 금지 영역 추가 (x55-60/y92-119 양면) + Q1 = SUD50P06-15-GE3 확정
Parts:
- Q1: value Q_PMOS_GDS -> SUD50P06-15-GE3
Changed lines of the file:
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@@
 	)
 	(junction
+		(at 287.02 50.8)
+		(diameter 0)
+		(color 0 0 0 0)
+	)
+	(junction
 		(at 289.56 78.74)
 		(diameter 0)
@@
 	(symbol
 		(lib_id "power:PWR_FLAG")
+		(at 287.02 50.8 0)
+		(unit 1)
+		(body_style 1)
+		(exclude_from_sim no)
+		(in_bom yes)
+		(on_board yes)
+		(in_pos_files yes)
+		(dnp no)
+		(fields_autoplaced yes)
+		(property "Reference" "#FLG03"
+			(at 287.02 48 0)
+			(hide yes)
+			(show_name no)
+			(do_not_autoplace no)
+			(effects
+				(font
+					(size 1.27 1.27)
+				)
+			)
+		)
+		(property "Value" "PWR_FLAG"
+			(at 287.02 48 90)
+			(show_name no)
+			(do_not_autoplace no)
+			(effects
+				(font
+					(size 1.27 1.27)
+				)
+				(justify left)
+			)
+		)
+		(property "Footprint" ""
+			(at 287.02 48 0)
+			(hide yes)
+			(show_name no)
+			(do_not_autoplace no)
+			(effects
+				(font
+					(size 1.27 1.27)
+				)
+			)
+		)
+		(property "Datasheet" ""
+			(at 287.02 48 0)
+			(hide yes)
+			(show_name no)
+			(do_not_autoplace no)
+			(effects
+				(font
+					(size 1.27 1.27)
+				)
+			)
+		)
+		(property "Description" "Special symbol for telling ERC where power comes from"
+			(at 287.02 48 0)
+			(hide yes)
+			(show_name no)
+			(do_not_autoplace no)
+			(effects
+				(font
+					(size 1.27 1.27)
+				)
+			)
+		)
+		(pin "1"
+		)
+		(instances
+			(project "OBD_CAN_ESP32_V2"
+				(path "/d818bd00-b54e-48fd-8a08-8c2bd25151ea"
+					(reference "#FLG03")
+					(unit 1)
+				)
+			)
+		)
+	)
+	(symbol
+		(lib_id "power:PWR_FLAG")
 		(at 152.4 181.61 270)
 		(unit 1)
@@
 			)
 		)
-		(property "Value" "Q_PMOS_GDS"
+		(property "Value" "SUD50P06-15-GE3"
 			(at 144.78 57.15 90)
 			(show_name no)
@@
 		)
 	)
-	(symbol
-		(lib_id "power:PWR_FLAG")
-		(at 287.02 50.8 0)
-		(unit 1)
-		(body_style 1)
-		(exclude_from_sim no)
-		(in_bom yes)
-		(on_board yes)
-		(in_pos_files yes)
-		(dnp no)
-		(fields_autoplaced yes)
-		(property "Reference" "#FLG03"
-			(at 287.02 48 0)
-			(hide yes)
-			(show_name no)
-			(do_not_autoplace no)
-			(effects
-				(font
-					(size 1.27 1.27)
-				)
-			)
-		)
-		(property "Value" "PWR_FLAG"
-			(at 287.02 48 90)
-			(show_name no)
-			(do_not_autoplace no)
-			(effects
-				(font
-					(size 1.27 1.27)
-				)
-				(justify left)
-			)
-		)
-		(property "Footprint" ""
-			(at 287.02 48 0)
-			(hide yes)
-			(show_name no)
-			(do_not_autoplace no)
-			(effects
-				(font
-					(size 1.27 1.27)
-				)
-			)
-		)
-		(property "Datasheet" ""
-			(at 287.02 48 0)
-			(hide yes)
-			(show_name no)
-			(do_not_autoplace no)
-			(effects
-				(font
-					(size 1.27 1.27)
-				)
-			)
-		)
-		(property "Description" "Special symbol for telling ERC where power comes from"
-			(at 287.02 48 0)
-			(hide yes)
-			(show_name no)
-			(do_not_autoplace no)
-			(effects
-				(font
-					(size 1.27 1.27)
-				)
-			)
-		)
-		(pin "1"
-		)
-		(instances
-			(project "OBD_CAN_ESP32_V2"
-				(path "/d818bd00-b54e-48fd-8a08-8c2bd25151ea"
-					(reference "#FLG03")
-					(unit 1)
-				)
-			)
-		)
-	)
-	(junction
-		(at 287.02 50.8)
-		(diameter 0)
-		(color 0 0 0 0)
-	)
-(sheet_instances
+	(sheet_instances
 		(path "/"
 			(page "1")
