File: hardware/OBD_CAN_ESP32_V2/OBD_CAN_ESP32_V2.kicad_pcb (KiCad board)
At the start: 2 copper layers, 64 x 36 mm, 39 parts, among them J1 OBD-II INPUT, J3 ESP32_S3_DEVKITC_J1, J4 ESP32_S3_DEVKITC_J3, Q1 Q_PMOS_GDS, U1 SN65HVD230, U2 TPS54360BDDA

Commit message: V2 PCB 배선 완료: 자동배선 + 미연결 13건 전량 수정 (GND 존 솔리드 연결, 스티칭 비아 8, D1 패드 정규화)
Routing:
- net /CAN_H: track 0.00 -> 142.6 mm, vias 0 -> 1
- net /CAN_L: track 0.00 -> 131.3 mm, vias 0 -> 1
- net /VBAT_PROTECTED: track 0.00 -> 98.5 mm, vias 0 -> 3
- net /+5V: track 0.00 -> 85.3 mm, vias 0 -> 3
- net /VBAT_FUSED: track 0.00 -> 65.0 mm, vias 0 -> 2
- net /CHASSIS_GND: track 0.00 -> 62.9 mm, vias 0 -> 1
- net /VBAT_OBD: track 0.00 -> 57.4 mm
- net /+3V3: track 0.00 -> 41.3 mm, vias 0 -> 1
- net /CAN_TX: track 0.00 -> 40.4 mm, vias 0 -> 2
- net /CAN_RX: track 0.00 -> 34.7 mm
- net Net-(D2-A): track 0.00 -> 24.7 mm, vias 0 -> 1
- net Net-(U2-FB): track 0.00 -> 23.3 mm
- net Net-(D10-K): track 0.00 -> 12.3 mm
- net Net-(U2-COMP): track 0.00 -> 11.2 mm
- net Net-(U2-RT/CLK): track 0.00 -> 9.58 mm
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
Commit message: V2 PCB: 배선 완료 (오류 0/미연결 0) + 끊긴 배선 꼬리 6개 정리
Routing:
- net Net-(D2-A): track 24.7 -> 18.0 mm
- net /+5V: track 85.3 -> 79.9 mm
- net /VBAT_FUSED: track 65.0 -> 60.1 mm
- net /CAN_TX: track 40.4 -> 37.0 mm
- net /VBAT_PROTECTED: track 98.5 -> 97.1 mm
